File: Magdamit_EE_201L_Project.kicad_pcb (KiCad board)
At the start: 2 copper layers, 125 x 77 mm, 63 parts, among them J1 Screw_Terminal_01x02, J2 Screw_Terminal_01x02, J3 Screw_Terminal_01x02

Commit message: 9.1.2025
Other:
- board text added: "BS ECE - 2A"
- board text removed: "ROVIC MAGDAMIT - BS ECE"
Changed lines of the file:
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@@
 		)
 	)
-	(gr_text "ROVIC MAGDAMIT - BS ECE"
+	(gr_text "BS ECE - 2A"
 		(at 35 105.5 0)
 		(layer "F.SilkS")

Commit message: 10.1.2025
Parts:
- removed Scan for GitHub repo: LOGO, QR:qr
- added Scan for Github Repo: LOGO, QR:qr_v2, F.Cu at (113.0, 126.5)
- moved +TP_R10 54.3 mm to (149.0, 117.5)
- moved +TP_R11 54.3 mm to (183.2, 72.5)
- moved +TP_R12 54.3 mm to (183.2, 87.5)
- moved +TP_R13 54.3 mm to (184.3, 100.1)
- moved +TP_R13-R15 54.3 mm to (193.5, 123.0)
- moved +TP_R14 54.3 mm to (184.3, 107.4)
- moved +TP_R15 54.3 mm to (184.3, 114.3)
- moved +TP_R6 54.3 mm to (149.0, 77.5)
- moved +TP_R7 54.3 mm to (149.0, 87.2)
- moved +TP_R8 54.3 mm to (149.0, 97.2)
- moved +TP_R9 54.3 mm to (149.0, 107.5)
- moved -TP 54.3 mm to (136.0, 73.2)
- moved -TP 54.3 mm to (173.8, 123.0)
- moved -TP_R11 54.3 mm to (183.2, 78.3)
- moved -TP_R12 54.3 mm to (183.2, 93.3)
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Other:
- board text added: "+9V"
- board text added: "+9v"
- board text added: "BS ECE - 2A @2025-2026"
- board text added: "Collaboration: OKSIJEAN Domingo, Andre Marick C. Lauglaug, Jhonas G. Magdamit, Rovic B. Magdaraog, John Paul M. Tabios, Gean G."
- board text removed: "+VCC"
- board text removed: "BS ECE - 2A"
