File: Magdamit_EE_201L_Project.kicad_sch (KiCad schematic)
At the start: 61 parts, among them J1 Screw_Terminal_01x02, J2 Screw_Terminal_01x02, J3 Screw_Terminal_01x02, SW1 SW_SPST, SW10 SW_SPST, SW11 SW_SPST, SW12 SW_SPST, SW13 SW_SPST, SW14 SW_SPST, SW2 SW_SPST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

Commit message: 10.1.2025
Parts:
- R1, R11, R6: value 330R -> 1K
- R12, R2, R7: value 470R -> 2K
- R13, R3, R8: value 510R -> 2.2K
- R14, R4, R9: value 1K -> 3.3K
Changed lines of the file:
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@@
 			)
 		)
-		(property "Value" "330R"
+		(property "Value" "1K"
 			(at 38.1 101.5999 0)
 			(effects
@@
 			)
 		)
-		(property "Value" "510R"
+		(property "Value" "2.2K"
 			(at 78.74 33.02 90)
 			(effects
@@
 			)
 		)
-		(property "Value" "1K"
+		(property "Value" "3.3K"
 			(at 110.49 166.3699 0)
 			(effects
@@
 			)
 		)
-		(property "Value" "330R"
+		(property "Value" "1K"
 			(at 30.48 137.16 90)
 			(effects
@@
 			)
 		)
-		(property "Value" "470R"
+		(property "Value" "2K"
 			(at 57.15 101.5999 0)
 			(effects
@@
 		(on_board yes)
 		(dnp no)
-		(fields_autoplaced yes)
 		(property "Reference" "SW1"
 			(at 40.64 30.48 0)
@@
 			)
 		)
-		(property "Value" "510R"
+		(property "Value" "2.2K"
 			(at 86.36 166.3699 0)
 			(effects
@@
 			)
 		)
-		(property "Value" "1K"
+		(property "Value" "3.3K"
 			(at 101.6 33.02 90)
 			(effects
@@
 			)
 		)
-		(property "Value" "470R"
+		(property "Value" "2K"
 			(at 50.8 33.02 90)
 			(effects
@@
 			)
 		)
-		(property "Value" "510R"
+		(property "Value" "2.2K"
 			(at 76.2 101.5999 0)
 			(effects
@@
 			)
 		)
-		(property "Value" "330R"
+		(property "Value" "1K"
 			(at 29.21 33.02 90)
 			(effects
@@
 			)
 		)
-		(property "Value" "470R"
+		(property "Value" "2K"
 			(at 55.88 137.16 90)
 			(effects
@@
 			)
 		)
-		(property "Value" "1K"
+		(property "Value" "3.3K"
 			(at 93.98 101.5999 0)
 			(effects
