File: EE_201L_Project.kicad_sch (KiCad schematic)
At the start: 83 parts, among them J1 Screw_Terminal_01x02, J2 Screw_Terminal_01x02, J3 Screw_Terminal_01x02, Q1 BC547, Q2 BC547, Q3 BC547, Q4 BC547, Q5 BC547, SW1 SW_SPST, SW10 SW_SPST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

Commit message: 10.22.2025
Parts:
- R1, R11: value 1K -> 100R
- R12: value 2K -> 510R
- R13: value 2.2K -> 1K
- R14: value 3.3K -> 2K2
- R15: value 4K7 -> 3K3
- R17: value 220 -> 330
- R2: value 2K -> 100R
- R20, R23: value 5k -> 5K1
- R3: value 2.2K -> 100R
- R4: value 3.3K -> 100R
- R5: value 4K7 -> 100R
Changed lines of the file:
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@@
 			)
 		)
-		(property "Value" "5k"
+		(property "Value" "5K1"
 			(at 133.35 109.2199 0)
 			(effects
@@
 			)
 		)
-		(property "Value" "2.2K"
+		(property "Value" "100R"
 			(at 78.74 33.02 90)
 			(effects
@@
 			)
 		)
-		(property "Value" "3.3K"
+		(property "Value" "2K2"
 			(at 110.49 166.3699 0)
 			(effects
@@
 			)
 		)
-		(property "Value" "1K"
+		(property "Value" "100R"
 			(at 30.48 137.16 90)
 			(effects
@@
 			)
 		)
-		(property "Value" "220"
+		(property "Value" "330"
 			(at 63.5 90.1699 0)
 			(effects
@@
 			)
 		)
-		(property "Value" "5k"
+		(property "Value" "5K1"
 			(at 194.31 107.9499 0)
 			(effects
@@
 			)
 		)
-		(property "Value" "4K7"
+		(property "Value" "100R"
 			(at 124.46 33.02 90)
 			(effects
@@
 			)
 		)
-		(property "Value" "4K7"
+		(property "Value" "3K3"
 			(at 134.62 166.3699 0)
 			(effects
@@
 			)
 		)
-		(property "Value" "2.2K"
+		(property "Value" "1K"
 			(at 86.36 166.3699 0)
 			(effects
@@
 			)
 		)
-		(property "Value" "3.3K"
+		(property "Value" "100R"
 			(at 101.6 33.02 90)
 			(effects
@@
 			)
 		)
-		(property "Value" "2K"
+		(property "Value" "100R"
 			(at 50.8 33.02 90)
 			(effects
@@
 			)
 		)
-		(property "Value" "1K"
+		(property "Value" "100R"
 			(at 29.21 33.02 90)
 			(effects
@@
 			)
 		)
-		(property "Value" "2K"
+		(property "Value" "510R"
 			(at 55.88 137.16 90)
 			(effects

Commit message: 10.22.2025 --fixed
Parts:
- R2: value 100R -> 220R
- R3: value 100R -> 330R
- R4: value 100R -> 470R
- R5: value 100R -> 510R
Changed lines of the file:
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@@
 			)
 		)
-		(property "Value" "100R"
+		(property "Value" "330R"
 			(at 78.74 33.02 90)
 			(effects
@@
 			)
 		)
-		(property "Value" "100R"
+		(property "Value" "510R"
 			(at 124.46 33.02 90)
 			(effects
@@
 			)
 		)
-		(property "Value" "100R"
+		(property "Value" "470R"
 			(at 101.6 33.02 90)
 			(effects
@@
 			)
 		)
-		(property "Value" "100R"
+		(property "Value" "220R"
 			(at 50.8 33.02 90)
 			(effects
